File: keyboards/alps75-zug/pcb/board/Quanta75_BareRP2040_JLCPCBAoptimized.kicad_pcb (KiCad board)
At the start: 2 copper layers, 320.7 x 158.3 mm, 276 parts, among them J1 USB_C_Receptacle_USB2.0, J10 Conn_01x05_Socket GPIOs, J2 Conn_01x02_Socket VBUS 5V, J3 Conn_01x02_Socket 3V3, J5 Conn_01x04_Socket SWD, J6 USB_A_Receptacle_UBS2.0, J7 USB_C_Receptacle_USB2.0, J8 Conn_01x04_Socket I2C display, J9 USB_C_Receptacle_USB2.0, M2.5 MountingHole_2.7mm_M2.5_DIN96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, M5Hole MountingHole_5.3mm_M5, SW1 SW_Push, SW10 SW_Push, SW11 SW_Push, SW12 SW_Push, SW13 SW_Push, SW14 SW_Push, SW15 SW_Push, SW16 SW_Push, SW17 SW_Push, SW18 SW_Push, SW19 SW_Push, SW2 SW_Push, SW20 SW_Push, SW21 SW_Push, SW22 SW_Push, SW23 SW_Push, SW24 SW_Push, SW25 SW_Push, SW26 SW_Push, SW27 SW_Push, SW28 SW_Push, SW29 SW_Push, SW3 SW_Push, SW30 SW_Push, SW31 SW_Push, SW32 SW_Push, SW33 SW_Push, SW34 SW_Push, SW35 SW_Push, SW36 SW_Push, SW37 SW_Push, SW38 SW_Push, SW39 SW_Push, SW4 SW_Push, SW40 SW_Push, SW41 SW_Push, SW42 SW_Push, SW43 SW_Push, SW44 SW_Push, SW45 SW_Push, SW46 SW_Push, SW47 SW_Push, SW48 SW_Push, SW49 SW_Push, SW5 SW_Push, SW50 SW_Push, SW51 SW_Push, SW52 SW_Push, SW53 SW_Push, SW54 SW_Push, SW55 SW_Push, SW56 SW_Push, SW57 SW_Push, SW58 SW_Push, SW59 SW_Push, SW6 SW_Push, SW60 SW_Push, SW61 SW_Push, SW62 SW_Push, SW63 SW_Push, SW64 SW_Push, SW65 SW_Push, SW66 SW_Push, SW67 SW_Push, SW68 SW_Push, SW69 SW_Push, SW7 SW_Push, SW70 SW_Push, SW71 SW_Push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

Commit message: Strip Cherry-style spacebar stabilizer footprint (no net impact)
Quanta75's 6.25u spacebar carries a PCM_Mounting_Keyboard_Stabilizer:
Stabilizer_Cherry_MX_6.25u footprint (Cherry clip-in stab cutout, all
pads non-plated/no net). Vintage Alps boards use different wire-stab
hardware with different mounting geometry, and Decision: stabilizers
is still reopened/unresolved, so removed rather than carried forward
incorrectly. Zero routing/electrical impact (mechanical-only footprint).

Per [Task: fork Quanta75 bare-RP2040 PCB and adapt to Alps 75% ANSI layout](https://github.com/bertrandvidal/stuff/issues/24) —
the spacebar switch footprint itself still needs its own Alps swap and
will need real stabilizer mounting once Decision: stabilizers closes.
Parts:
- removed 6.25u stabilizer: Stabilizer_Cherry_MX_6.25u, PCM_Mounting_Keyboard_Stabilizer:Stabilizer_Cherry_MX_6.25u
