File: keyboards/alps75-zug/pcb/board/Quanta75_BareRP2040_JLCPCBAoptimized.kicad_pcb (KiCad board)
At the start: 2 copper layers, 320.7 x 158.3 mm, 275 parts, among them J1 USB_C_Receptacle_USB2.0, J10 Conn_01x05_Socket GPIOs, J2 Conn_01x02_Socket VBUS 5V, J3 Conn_01x02_Socket 3V3, J5 Conn_01x04_Socket SWD, J6 USB_A_Receptacle_UBS2.0, J7 USB_C_Receptacle_USB2.0, J8 Conn_01x04_Socket I2C display, J9 USB_C_Receptacle_USB2.0, M2.5 MountingHole_2.7mm_M2.5_DIN96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, M5Hole MountingHole_5.3mm_M5, SW1 SW_Push, SW10 SW_Push, SW11 SW_Push, SW12 SW_Push, SW13 SW_Push, SW14 SW_Push, SW15 SW_Push, SW16 SW_Push, SW17 SW_Push, SW18 SW_Push, SW19 SW_Push, SW2 SW_Push, SW20 SW_Push, SW21 SW_Push, SW22 SW_Push, SW23 SW_Push, SW24 SW_Push, SW25 SW_Push, SW26 SW_Push, SW27 SW_Push, SW28 SW_Push, SW29 SW_Push, SW3 SW_Push, SW30 SW_Push, SW31 SW_Push, SW32 SW_Push, SW33 SW_Push, SW34 SW_Push, SW35 SW_Push, SW36 SW_Push, SW37 SW_Push, SW38 SW_Push, SW39 SW_Push, SW4 SW_Push, SW40 SW_Push, SW41 SW_Push, SW42 SW_Push, SW43 SW_Push, SW44 SW_Push, SW45 SW_Push, SW46 SW_Push, SW47 SW_Push, SW48 SW_Push, SW49 SW_Push, SW5 SW_Push, SW50 SW_Push, SW51 SW_Push, SW52 SW_Push, SW53 SW_Push, SW54 SW_Push, SW55 SW_Push, SW56 SW_Push, SW57 SW_Push, SW58 SW_Push, SW59 SW_Push, SW6 SW_Push, SW60 SW_Push, SW61 SW_Push, SW62 SW_Push, SW63 SW_Push, SW64 SW_Push, SW65 SW_Push, SW66 SW_Push, SW67 SW_Push, SW68 SW_Push, SW69 SW_Push, SW7 SW_Push, SW70 SW_Push, SW71 SW_Push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

Commit message: Swap PCB switch footprints Cherry MX -> Alps_Solderable (81 of 82)
PCB-side half of the footprint swap for Task: fork Quanta75 bare-RP2040
PCB and adapt to Alps 75% ANSI layout. All 81 non-ISO switches: lib_id,
silkscreen graphics, and pads replaced with the matching Alps_Solderable
size, net assignments carried over by pad number (verified against the
schematic's already-swapped Footprint properties). No 3D model kept --
ai03/MX_V2 ships none for Alps_Solderable, and pointing at the old
Cherry .wrl would show the wrong switch shape.

Electrically correct (pad->net mapping right), but NOT physically
routed: Alps pin spacing differs enough from Cherry MX's that the new
pad position collides with pre-existing copper at 37 of 81 switches,
confirmed with kicad-cli pcb drc on the swap alone, before touching any
trace. Tried two automated trace fixes (translate touching endpoints;
delete and leave unrouted) -- translating created new shorts (naive
endpoint moves have no pathfinding), deleting is honest but doesn't
resolve the 37 collisions either. Both need visual judgment a text
edit can't safely substitute for.

Traces left untouched (still pointing at the old, now-vacated Cherry
pad positions) as the least-invasive starting point for manual
reroute. Full handoff checklist, exact switch list, and DRC baseline
to route back down to: pcb/board/REROUTE-CHECKLIST.md.

Also stops tracking the per-machine *.kicad_prl view-state file
(kicad-cli rewrites it on every invocation; not real project content).
Parts:
- SW1, SW10, SW11, SW12, SW13, SW14, SW15, SW16, SW17, SW18, SW19, SW2, SW20, SW21, SW22, SW23, SW24, SW25, SW26, SW28, SW3, SW30, SW31, SW32, SW33, SW34, SW35, SW36, SW37, SW38, SW39, SW4, SW40, SW41, SW43, SW45, SW46, SW47, SW48, SW49, SW5, SW50, SW51, SW52, SW53, SW54, SW55, SW56, SW57, SW59, SW6, SW60, SW61, SW62, SW63, SW64, SW65, SW66, SW67, SW68, SW69, SW7, SW71, SW72, SW77, SW78, SW79, SW8, SW80, SW81, SW82, SW9: footprint Button_Switch_Keyboard:SW_Cherry_MX_1.00u_PCB -> Alps_Solderable:Alps-Solderable-1U
- SW27: footprint Button_Switch_Keyboard:SW_Cherry_MX_2.00u_PCB -> Alps_Solderable:Alps-Solderable-2U
- SW29: footprint Button_Switch_Keyboard:SW_Cherry_MX_1.50u_PCB -> Alps_Solderable:Alps-Solderable-1.5U
- SW44, SW70: footprint Button_Switch_Keyboard:SW_Cherry_MX_1.75u_PCB -> Alps_Solderable:Alps-Solderable-1.75U
- SW58, SW73, SW74, SW75: footprint Button_Switch_Keyboard:SW_Cherry_MX_1.25u_PCB -> Alps_Solderable:Alps-Solderable-1.25U
- SW76: footprint PCM_Switch_Keyboard_Cherry_MX:SW_Cherry_MX_PCB_6.25u -> Alps_Solderable:Alps-Solderable-6.25U
