File: keyboards/alps75-zug/pcb/board/Quanta75_BareRP2040_JLCPCBAoptimized.kicad_sch (KiCad schematic)
At the start: 246 parts, among them J1 USB_C_Receptacle_USB2.0, J10 Conn_01x05_Socket GPIOs, J2 Conn_01x02_Socket VBUS 5V, J3 Conn_01x02_Socket 3V3, J5 Conn_01x04_Socket SWD, J6 USB_A_Receptacle_UBS2.0, J7 USB_C_Receptacle_USB2.0, J8 Conn_01x04_Socket I2C display, J9 USB_C_Receptacle_USB2.0, SW1 SW_Push, SW10 SW_Push, SW11 SW_Push, SW12 SW_Push, SW13 SW_Push, SW14 SW_Push, SW15 SW_Push, SW16 SW_Push, SW17 SW_Push, SW18 SW_Push, SW19 SW_Push, SW2 SW_Push, SW20 SW_Push, SW21 SW_Push, SW22 SW_Push, SW23 SW_Push, SW24 SW_Push, SW25 SW_Push, SW26 SW_Push, SW27 SW_Push, SW28 SW_Push, SW29 SW_Push, SW3 SW_Push, SW30 SW_Push, SW31 SW_Push, SW32 SW_Push, SW33 SW_Push, SW34 SW_Push, SW35 SW_Push, SW36 SW_Push, SW37 SW_Push, SW38 SW_Push, SW39 SW_Push, SW4 SW_Push, SW40 SW_Push, SW41 SW_Push, SW42 SW_Push, SW43 SW_Push, SW44 SW_Push, SW45 SW_Push, SW46 SW_Push, SW47 SW_Push, SW48 SW_Push, SW49 SW_Push, SW5 SW_Push, SW50 SW_Push, SW51 SW_Push, SW52 SW_Push, SW53 SW_Push, SW54 SW_Push, SW55 SW_Push, SW56 SW_Push, SW57 SW_Push, SW58 SW_Push, SW59 SW_Push, SW6 SW_Push, SW60 SW_Push, SW61 SW_Push, SW62 SW_Push, SW63 SW_Push, SW64 SW_Push, SW65 SW_Push, SW66 SW_Push, SW67 SW_Push, SW68 SW_Push, SW69 SW_Push, SW7 SW_Push, SW70 SW_Push, SW71 SW_Push, SW72 SW_Push, SW73 SW_Push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

Commit message: Fix Alps footprint swap: correct placement and pad numbering
The previous swap (058b1e5) left 37 of 81 switches apparently colliding
with Quanta75's row backbone, which looked like an inherent Alps/Cherry
incompatibility requiring manual rerouting. It wasn't. Three bugs:

1. KiCad's Button_Switch_Keyboard:SW_Cherry_MX_*_PCB footprints put
   their origin ON PAD 1, with the key centre at local (-2.54, 5.08);
   ai03's Alps footprints put their origin ON THE KEY CENTRE. Reusing
   the Cherry (at ...) verbatim moved every switch 5.68mm diagonally
   off the keycap grid.

2. The two libraries number their pads on opposite sides of the switch
   (Cherry pad 1 = upper right, ai03 pad 1 = upper left), so carrying
   nets across by pad number sent each one to the hole on the far side
   -- a 5.1mm / 6.6mm jump. That, not the switch geometry, is what hit
   the row backbone.

3. DRC had been run without --refill-zones, so a stale GND pour added
   several hundred phantom violations against switch pads.

Corrected here: switches placed at their true key centres (verified
identical to upstream Quanta75 across all 82, so keycap fit is
unchanged), and pad numbering reconciled via a derived footprint
library rather than by editing the schematic. A keyswitch is a
non-polar SPST contact, so renumbering its pads changes nothing
electrically; the diode carries the polarity.

Each net now lands 0.58mm and 1.96mm from copper it already reaches,
so reconnection is one uniform ~2mm stub per switch -- 86 segments,
all generated mechanically, no interactive routing.

kicad-cli pcb drc --refill-zones: 284 violations vs. upstream's 302.
No new shorting items, no new clearance violations. The one genuinely
new item is a dangling Net-(D76-A) track at SW76, the ISO Enter key,
which the ANSI reshape removes anyway.

REROUTE-CHECKLIST.md is deleted: its 37-switch list described damage
from the bad swap, not real geometry.

Refs: https://github.com/bertrandvidal/stuff/issues/24

Co-Authored-By: Cl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
Parts:
- SW1, SW10, SW11, SW12, SW13, SW14, SW15, SW16, SW17, SW18, SW19, SW2, SW20, SW21, SW22, SW23, SW24, SW25, SW26, SW28, SW3, SW30, SW31, SW32, SW33, SW34, SW35, SW36, SW37, SW38, SW39, SW4, SW40, SW41, SW43, SW45, SW46, SW47, SW48, SW49, SW5, SW50, SW51, SW52, SW53, SW54, SW55, SW56, SW57, SW59, SW6, SW60, SW61, SW62, SW63, SW64, SW65, SW66, SW67, SW68, SW69, SW7, SW71, SW72, SW77, SW78, SW79, SW8, SW80, SW81, SW82, SW9: footprint Alps_Solderable:Alps-Solderable-1U -> Alps_Solderable_MXPadOrder:Alps-Solderable-1U
- SW27: footprint Alps_Solderable:Alps-Solderable-2U -> Alps_Solderable_MXPadOrder:Alps-Solderable-2U
- SW29: footprint Alps_Solderable:Alps-Solderable-1.5U -> Alps_Solderable_MXPadOrder:Alps-Solderable-1.5U
- SW44, SW70: footprint Alps_Solderable:Alps-Solderable-1.75U -> Alps_Solderable_MXPadOrder:Alps-Solderable-1.75U
- SW58, SW73, SW74, SW75: footprint Alps_Solderable:Alps-Solderable-1.25U -> Alps_Solderable_MXPadOrder:Alps-Solderable-1.25U
- SW76: footprint Alps_Solderable:Alps-Solderable-6.25U -> Alps_Solderable_MXPadOrder:Alps-Solderable-6.25U
