File: keyboards/alps75-zug/pcb/alps75-zug.kicad_pcb (KiCad board)
At the start: 2 copper layers, 340.3 x 130.7 mm, 184 parts, among them SW1 SW_Push, SW10 SW_Push, SW11 SW_Push, SW12 SW_Push, SW13 SW_Push, SW14 SW_Push, SW15 SW_Push, SW16 SW_Push, SW17 SW_Push, SW18 SW_Push, SW19 SW_Push, SW2 SW_Push, SW20 SW_Push, SW21 SW_Push, SW22 SW_Push, SW23 SW_Push, SW24 SW_Push, SW25 SW_Push, SW26 SW_Push, SW27 SW_Push, SW28 SW_Push, SW29 SW_Push, SW3 SW_Push, SW30 SW_Push, SW31 SW_Push, SW32 SW_Push, SW33 SW_Push, SW34 SW_Push, SW35 SW_Push, SW36 SW_Push, SW37 SW_Push, SW38 SW_Push, SW39 SW_Push, SW4 SW_Push, SW40 SW_Push, SW41 SW_Push, SW42 SW_Push, SW43 SW_Push, SW44 SW_Push, SW45 SW_Push, SW46 SW_Push, SW47 SW_Push, SW48 SW_Push, SW49 SW_Push, SW5 SW_Push, SW50 SW_Push, SW51 SW_Push, SW52 SW_Push, SW53 SW_Push, SW54 SW_Push, SW55 SW_Push, SW56 SW_Push, SW57 SW_Push, SW58 SW_Push, SW59 SW_Push, SW6 SW_Push, SW60 SW_Push, SW61 SW_Push, SW62 SW_Push, SW63 SW_Push, SW64 SW_Push, SW65 SW_Push, SW66 SW_Push, SW67 SW_Push, SW68 SW_Push, SW69 SW_Push, SW7 SW_Push, SW70 SW_Push, SW71 SW_Push, SW72 SW_Push, SW73 SW_Push, SW74 SW_Push, SW75 SW_Push, SW76 SW_Push, SW77 SW_Push, SW78 SW_Push, SW79 SW_Push, SW8 SW_Push, SW80 SW_Push, SW81 SW_Push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

Commit message: Add RP2040 (U1) to alps75-zug and wire the key matrix to it
Schematic: add an RP2040 (QFN-56 7x7mm) with the 6 ROW and 17 COL
global labels attached to its GPIOs, so every matrix net now ends on
U1. Power, USB, QSPI flash, crystal, SWD and RUN pins are still
unconnected. The 8 Mechanical:MountingHole symbols are removed.

PCB, after update from schematic:
- U1 placed on F.Cu at (296.275, 227.6), below the key area, with the
  ROW/COL fan-out routed (129 new segments, 6 vias on the ROW nets).
- Mounting holes H1-H8 removed, following the schematic.
- Rounded Edge.Cuts outline replaced by a 358 x 172.5 mm rectangle
  enlarged to take the controller area.
- Footprints and existing tracks moved by (-8.5, +51.3) mm.

Also picks up the local KiCad view state (.kicad_prl) and U1 in the
used designators (.kicad_pro).

Co-Authored-By: Claude Opus 5 <noreply@anthropic.com>
Parts:
- removed H1, H2, H3, H4, H5, H6, H7, H8: MountingHole_3.2mm_M3, MountingHole:MountingHole_3.2mm_M3
- added U1: RP2040, Package_DFN_QFN:QFN-56-1EP_7x7mm_P0.4mm_EP3.2x3.2mm, F.Cu at (306.8, 240.6)
- moved D1 64.3 mm to (146.2, 149.6)
- moved D10 64.3 mm to (317.7, 149.6)
- moved D11 64.3 mm to (336.7, 149.6)
- moved D12 64.3 mm to (355.8, 149.6)
- moved D13 64.3 mm to (374.8, 149.6)
- moved D14 64.3 mm to (393.9, 149.6)
- moved D15 64.3 mm to (412.9, 149.6)
- moved D16 64.3 mm to (432.0, 149.6)
- moved D17 64.3 mm to (451.0, 149.6)
- moved D2 64.3 mm to (165.3, 149.6)
- moved D3 64.3 mm to (184.3, 149.6)
- moved D4 64.3 mm to (203.4, 149.6)
- moved D5 64.3 mm to (222.4, 149.6)
- moved D6 64.3 mm to (241.5, 149.6)
- moved D7 64.3 mm to (260.5, 149.6)
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Connections:
- SW83 pad 1: COL10 -> COL11
Routing:
- net ROW0: track 304.8 -> 535.1 mm, vias 0 -> 1
- net ROW1: track 304.8 -> 514.9 mm, vias 0 -> 1
- net ROW2: track 300.0 -> 489.7 mm, vias 0 -> 1
- net ROW3: track 297.7 -> 466.4 mm, vias 0 -> 1
- net COL0: track 103.1 -> 266.4 mm
- net COL2: track 86.1 -> 227.3 mm
- net COL1: track 102.2 -> 238.9 mm
- net COL16: track 95.3 -> 230.0 mm
- net COL15: track 95.3 -> 210.7 mm
- net COL3: track 107.1 -> 217.5 mm
- net COL14: track 104.6 -> 200.7 mm
- net COL4: track 86.1 -> 180.5 mm
- net COL13: track 107.1 -> 184.0 mm
- net COL5: track 86.1 -> 162.0 mm
- net COL6: track 86.1 -> 151.5 mm
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Other:
- board size 340.3 x 130.7 mm -> 358 x 172.5 mm
