File: keyboards/alps75-zug/pcb/v0.1/alps75-zug.kicad_sch (KiCad schematic)
At the start: 177 parts, among them SW1 SW_Push, SW10 SW_Push, SW11 SW_Push, SW12 SW_Push, SW13 SW_Push, SW14 SW_Push, SW15 SW_Push, SW16 SW_Push, SW17 SW_Push, SW18 SW_Push, SW19 SW_Push, SW2 SW_Push, SW20 SW_Push, SW21 SW_Push, SW22 SW_Push, SW23 SW_Push, SW24 SW_Push, SW25 SW_Push, SW26 SW_Push, SW27 SW_Push, SW28 SW_Push, SW29 SW_Push, SW3 SW_Push, SW30 SW_Push, SW31 SW_Push, SW32 SW_Push, SW33 SW_Push, SW34 SW_Push, SW35 SW_Push, SW36 SW_Push, SW37 SW_Push, SW38 SW_Push, SW39 SW_Push, SW4 SW_Push, SW40 SW_Push, SW41 SW_Push, SW42 SW_Push, SW43 SW_Push, SW44 SW_Push, SW45 SW_Push, SW46 SW_Push, SW47 SW_Push, SW48 SW_Push, SW49 SW_Push, SW5 SW_Push, SW50 SW_Push, SW51 SW_Push, SW52 SW_Push, SW53 SW_Push, SW54 SW_Push, SW55 SW_Push, SW56 SW_Push, SW57 SW_Push, SW58 SW_Push, SW59 SW_Push, SW6 SW_Push, SW60 SW_Push, SW61 SW_Push, SW62 SW_Push, SW63 SW_Push, SW64 SW_Push, SW65 SW_Push, SW66 SW_Push, SW67 SW_Push, SW68 SW_Push, SW69 SW_Push, SW7 SW_Push, SW70 SW_Push, SW71 SW_Push, SW72 SW_Push, SW73 SW_Push, SW74 SW_Push, SW75 SW_Push, SW76 SW_Push, SW77 SW_Push, SW78 SW_Push, SW79 SW_Push, SW8 SW_Push, SW80 SW_Push, SW81 SW_Push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

Commit message: Rename to v0.1
Move the KiCad project to pcb/v0.1/ and the plate to plate/v0.1/, and
stamp v0.1 into the design files themselves.

Versioning by folder rather than by file basename keeps the KiCad
basename stable, so the 177 sheetfile references inside the board and
the filename keys in .kicad_pro / .kicad_prl need no rewriting now or at
any future rev bump. The next revision is a folder copy that leaves v0.1
intact beside it, matching how old-pcb/ already holds the previous
design.

Version now appears in:
- schematic title_block: added title, date and rev (v0.1), keeping the
  two kbplacer comments
- board title_block: added outright, the PCB had none at all
- KLE metadata notes in layout.json and pcb/v0.1/alps75-zug.json

The back silkscreen already read "alps75-zug - 2026 - v0.1" and is
unchanged. The version went in KLE meta.notes rather than meta.name
because KLE-NG derives the generated plate filename from name, which
would churn the basename on every regen.

Also corrects the plate header comment, which still claimed 2 mm
thickness after THICKNESS dropped to 1.8.

kicad-cli after the move reproduces the recorded baseline exactly: ERC
28 pin_not_connected, 6 power_pin_not_driven, 4 pin_not_driven, 1
unconnected_wire_endpoint; DRC 0 violations, 6 unconnected_items, 0
schematic parity issues. fp-lib-table resolves via ${KIPRJMOD} and
needed no edit.

Co-Authored-By: Claude Opus 5 <noreply@anthropic.com>
Other:
- title: (none) -> alps75-zug
Changed lines of the file:
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@@
 	(paper "A2")
 	(title_block
+		(title "alps75-zug")
+		(date "2026-09-17")
+		(rev "v0.1")
 		(comment 1 "https://github.com/adamws/kicad-kbplacer")
 		(comment 2 "Auto-generated with kicad-kbplacer, requires validation before production!")
