File: keyboards/alps75-zug/alps75-zug.kicad_pcb (KiCad board)
At the start: 2 copper layers, 176 parts, among them SW1 SW_Push, SW10 SW_Push, SW11 SW_Push, SW12 SW_Push, SW13 SW_Push, SW14 SW_Push, SW15 SW_Push, SW16 SW_Push, SW17 SW_Push, SW18 SW_Push, SW19 SW_Push, SW2 SW_Push, SW20 SW_Push, SW21 SW_Push, SW22 SW_Push, SW23 SW_Push, SW24 SW_Push, SW25 SW_Push, SW26 SW_Push, SW27 SW_Push, SW28 SW_Push, SW29 SW_Push, SW3 SW_Push, SW30 SW_Push, SW31 SW_Push, SW32 SW_Push, SW33 SW_Push, SW34 SW_Push, SW35 SW_Push, SW36 SW_Push, SW37 SW_Push, SW38 SW_Push, SW39 SW_Push, SW4 SW_Push, SW40 SW_Push, SW41 SW_Push, SW42 SW_Push, SW43 SW_Push, SW44 SW_Push, SW45 SW_Push, SW46 SW_Push, SW47 SW_Push, SW48 SW_Push, SW49 SW_Push, SW5 SW_Push, SW50 SW_Push, SW51 SW_Push, SW52 SW_Push, SW53 SW_Push, SW54 SW_Push, SW55 SW_Push, SW56 SW_Push, SW57 SW_Push, SW58 SW_Push, SW59 SW_Push, SW6 SW_Push, SW60 SW_Push, SW61 SW_Push, SW62 SW_Push, SW63 SW_Push, SW64 SW_Push, SW65 SW_Push, SW66 SW_Push, SW67 SW_Push, SW68 SW_Push, SW69 SW_Push, SW7 SW_Push, SW70 SW_Push, SW71 SW_Push, SW72 SW_Push, SW73 SW_Push, SW74 SW_Push, SW75 SW_Push, SW76 SW_Push, SW77 SW_Push, SW78 SW_Push, SW79 SW_Push, SW8 SW_Push, SW80 SW_Push, SW81 SW_Push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

Commit message: Resize schematic + PCB page to fit
Parts:
- moved D1 142.2 mm to (58.8, 126.2)
- moved D10 142.2 mm to (230.3, 126.2)
- moved D11 142.2 mm to (249.3, 126.2)
- moved D12 142.2 mm to (268.4, 126.2)
- moved D13 142.2 mm to (287.4, 126.2)
- moved D14 142.2 mm to (306.5, 126.2)
- moved D15 142.2 mm to (325.5, 126.2)
- moved D16 142.2 mm to (344.6, 126.2)
- moved D17 142.2 mm to (363.6, 126.2)
- moved D18 142.2 mm to (59.9, 154.3)
- moved D19 142.2 mm to (79.0, 154.3)
- moved D2 142.2 mm to (77.9, 126.2)
- moved D20 142.2 mm to (98.0, 154.3)
- moved D21 142.2 mm to (117.1, 154.3)
- moved D22 142.2 mm to (136.1, 154.3)
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
Commit message: Add a tab to the PCB to hold the Pico board
Parts:
- added U1: RaspberryPi_Pico, Module:RaspberryPi_Pico_SMD_HandSolder, B.Cu at (62.6, 109.5)
Other:
- board outline added: 332.6 x 139.1 mm

Commit message: Connected all diodes for F-keys + move COL14 wire out of way
Parts:
- moved U1 8.30 mm to (62.6, 101.2)
Routing:
- net ROW0: track 0.00 -> 497.8 mm
- net COL14: track 89.4 -> 95.6 mm
Other:
- board size 332.6 x 139.1 mm -> 332.6 x 147.5 mm

Commit message: Increase edge cuts to have more room to route
Parts:
- U1: moved to F.Cu
- turned U1 to 90 degrees
Other:
- board size 332.6 x 147.5 mm -> 335.4 x 156.5 mm

Commit message: Wire switches to MCU
PCB edges are updated to be the same on the side, cols wiring is from the F-key rows rather than from the bottom to shorten wiring, rows wiring from the right side of the PCB.
Connections:
- U1 pad 1: (no net) -> COL0
- U1 pad 10: (no net) -> COL7
- U1 pad 11: (no net) -> COL8
- U1 pad 12: (no net) -> COL9
- U1 pad 13: (no net) -> Net-(U1-GND-Pad13)
- U1 pad 14: (no net) -> COL10
- U1 pad 15: (no net) -> COL11
- U1 pad 16: (no net) -> COL12
- U1 pad 17: (no net) -> COL13
- U1 pad 18: (no net) -> Net-(U1-GND-Pad13)
- U1 pad 19: (no net) -> COL14
- U1 pad 2: (no net) -> COL1
- U1 pad 20: (no net) -> COL15
- U1 pad 21: (no net) -> COL16
- U1 pad 22: (no net) -> ROW0
- U1 pad 23: (no net) -> Net-(U1-GND-Pad13)
- U1 pad 24: (no net) -> ROW1
- U1 pad 25: (no net) -> ROW2
- U1 pad 26: (no net) -> ROW3
- U1 pad 27: (no net) -> ROW4
- U1 pad 28: (no net) -> Net-(U1-GND-Pad13)
- U1 pad 29: (no net) -> ROW5
- U1 pad 3: (no net) -> Net-(U1-GND-Pad13)
- U1 pad 30: (no net) -> unconnected-(U1-RUN-Pad30)
- U1 pad 31: (no net) -> unconnected-(U1-GPIO26_ADC0-Pad31)
- U1 pad 32: (no net) -> unconnected-(U1-GPIO27_ADC1-Pad32)
- U1 pad 33: (no net) -> unconnected-(U1-AGND-Pad33)
- U1 pad 34: (no net) -> unconnected-(U1-GPIO28_ADC2-Pad34)
- U1 pad 35: (no net) -> unconnected-(U1-ADC_VREF-Pad35)
- U1 pad 36: (no net) -> unconnected-(U1-3V3-Pad36)
- U1 pad 37: (no net) -> unconnected-(U1-3V3_EN-Pad37)
- U1 pad 38: (no net) -> Net-(U1-GND-Pad13)
- U1 pad 39: (no net) -> unconnected-(U1-VSYS-Pad39)
- U1 pad 4: (no net) -> COL2
- U1 pad 40: (no net) -> unconnected-(U1-VBUS-Pad40)
- U1 pad 5: (no net) -> COL3
- U1 pad 6: (no net) -> COL4
- U1 pad 7: (no net) -> COL5
- U1 pad 8: (no net) -> Net-(U1-GND-Pad13)
- U1 pad 9: (no net) -> COL6
- U1 pad D1: (no net) -> unconnected-(U1-SWCLK-PadD1)
- U1 pad D2: (no net) -> Net-(U1-GND-Pad13)
- U1 pad D3: (no net) -> unconnected-(U1-SWDIO-PadD3)
Routing:
- net ROW5: track 300.0 -> 762.2 mm, vias 0 -> 1
- net ROW4: track 292.9 -> 727.9 mm, vias 0 -> 1
- net ROW3: track 297.7 -> 708.1 mm, vias 0 -> 1
- net ROW2: track 300.0 -> 685.9 mm, vias 0 -> 1
- net ROW1: track 304.8 -> 666.0 mm, vias 0 -> 1
- net COL16: track 89.4 -> 406.5 mm
- net COL15: track 89.4 -> 363.6 mm
- net COL14: track 95.6 -> 353.3 mm
- net COL13: track 101.2 -> 345.0 mm
- net COL12: track 97.3 -> 324.5 mm
- net COL11: track 80.2 -> 291.0 mm
- net COL10: track 104.2 -> 298.4 mm
- net COL9: track 80.2 -> 260.5 mm
- net COL8: track 80.2 -> 244.0 mm
- net COL7: track 101.2 -> 248.5 mm
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Other:
- board size 335.4 x 156.5 mm -> 340.3 x 161.5 mm

Commit message: Tighten the Pico's tab to be trimmed to the copper
Other:
- board size 340.3 x 161.5 mm -> 340.3 x 159.9 mm
Changed lines of the file:
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@@
 	)
 	(gr_arc
-		(start 37.08 81.5)
-		(mid 37.3729 80.7929)
-		(end 38.08 80.5)
+		(start 37.08 83.09)
+		(mid 37.3729 82.3829)
+		(end 38.08 82.09)
 		(stroke
 			(width 0.05)
@@
 	)
 	(gr_line
-		(start 38.08 80.5)
-		(end 129 80.5)
+		(start 38.08 82.09)
+		(end 97.91 82.09)
 		(stroke
 			(width 0.05)
@@
 	)
 	(gr_arc
-		(start 129 80.5)
-		(mid 129.7071 80.7929)
-		(end 130 81.5)
+		(start 97.91 82.09)
+		(mid 98.6171 82.3829)
+		(end 98.91 83.09)
 		(stroke
 			(width 0.05)
@@
 	)
 	(gr_line
-		(start 130 81.5)
-		(end 130 115)
+		(start 98.91 83.09)
+		(end 98.91 115)
 		(stroke
 			(width 0.05)
@@
 	)
 	(gr_arc
-		(start 130 115)
-		(mid 130.2929 115.7071)
-		(end 131 116)
+		(start 98.91 115)
+		(mid 99.2029 115.7071)
+		(end 99.91 116)
 		(stroke
 			(width 0.05)
@@
 	)
 	(gr_line
-		(start 131 116)
+		(start 99.91 116)
 		(end 376.3825 116)
 		(stroke
@@
 	(gr_line
 		(start 37.08 241)
-		(end 37.08 81.5)
+		(end 37.08 83.09)
 		(stroke
 			(width 0.05)

Commit message: Move pico as low as possible + reroute all copper
Parts:
- moved U1 7.20 mm to (62.6, 108.4)
Routing:
- net ROW2: track 685.9 -> 678.7 mm
- net COL15: track 363.6 -> 356.4 mm
- net ROW4: track 727.9 -> 720.7 mm
- net ROW3: track 708.1 -> 700.9 mm
- net COL3: track 185.0 -> 177.8 mm
- net COL14: track 353.3 -> 346.1 mm
- net COL13: track 345.0 -> 337.8 mm
- net COL11: track 291.0 -> 283.8 mm
- net COL9: track 260.5 -> 253.3 mm
- net COL8: track 244.0 -> 236.8 mm
- net COL7: track 248.5 -> 241.3 mm
- net COL4: track 180.5 -> 173.3 mm
- net COL0: track 134.0 -> 126.8 mm
- net COL6: track 210.9 -> 203.7 mm
- net COL5: track 197.0 -> 189.8 mm
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Other:
- board size 340.3 x 159.9 mm -> 340.3 x 152.7 mm
- board text added: "alps75-zug - v0.1 - Bert Vidal - 2026"

Commit message: Connect GND pins via F.Cu
Routing:
- net Net-(U1-GND-Pad13): track 0.00 -> 115.2 mm
Changed lines of the file:
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@@
 		(net "Net-(D73-A)")
+	)
+	(segment
+		(start 43.53 98.71)
+		(end 43.53 104)
+		(width 0.2)
+		(layer "F.Cu")
+		(net "Net-(U1-GND-Pad13)")
+	)
+	(segment
+		(start 43.53 104)
+		(end 43.53 118.09)
+		(width 0.2)
+		(layer "F.Cu")
+		(net "Net-(U1-GND-Pad13)")
+	)
+	(segment
+		(start 68.93 98.71)
+		(end 68.93 104)
+		(width 0.2)
+		(layer "F.Cu")
+		(net "Net-(U1-GND-Pad13)")
+	)
+	(segment
+		(start 68.93 104)
+		(end 68.93 118.09)
+		(width 0.2)
+		(layer "F.Cu")
+		(net "Net-(U1-GND-Pad13)")
+	)
+	(segment
+		(start 81.63 98.71)
+		(end 81.63 104)
+		(width 0.2)
+		(layer "F.Cu")
+		(net "Net-(U1-GND-Pad13)")
+	)
+	(segment
+		(start 81.63 104)
+		(end 81.63 108.4)
+		(width 0.2)
+		(layer "F.Cu")
+		(net "Net-(U1-GND-Pad13)")
+	)
+	(segment
+		(start 81.63 108.4)
+		(end 81.63 118.09)
+		(width 0.2)
+		(layer "F.Cu")
+		(net "Net-(U1-GND-Pad13)")
+	)
+	(segment
+		(start 56.23 104)
+		(end 56.23 118.09)
+		(width 0.2)
+		(layer "F.Cu")
+		(net "Net-(U1-GND-Pad13)")
+	)
+	(segment
+		(start 43.53 104)
+		(end 56.23 104)
+		(width 0.2)
+		(layer "F.Cu")
+		(net "Net-(U1-GND-Pad13)")
+	)
+	(segment
+		(start 56.23 104)
+		(end 68.93 104)
+		(width 0.2)
+		(layer "F.Cu")
+		(net "Net-(U1-GND-Pad13)")
+	)
+	(segment
+		(start 68.93 104)
+		(end 81.63 104)
+		(width 0.2)
+		(layer "F.Cu")
+		(net "Net-(U1-GND-Pad13)")
+	)
+	(segment
+		(start 81.63 108.4)
+		(end 86.48 108.4)
+		(width 0.2)
+		(layer "F.Cu")
+		(net "Net-(U1-GND-Pad13)")
 	)
 	(embedded_fonts no)
