File: keyboards/alps75-zug/alps75-zug.kicad_pcb (KiCad board)
At the start: 2 copper layers, 328 x 147.2 mm, 177 parts, among them SW1 SW_Push, SW10 SW_Push, SW11 SW_Push, SW12 SW_Push, SW13 SW_Push, SW14 SW_Push, SW15 SW_Push, SW16 SW_Push, SW17 SW_Push, SW18 SW_Push, SW19 SW_Push, SW2 SW_Push, SW20 SW_Push, SW21 SW_Push, SW22 SW_Push, SW23 SW_Push, SW24 SW_Push, SW25 SW_Push, SW26 SW_Push, SW27 SW_Push, SW28 SW_Push, SW29 SW_Push, SW3 SW_Push, SW30 SW_Push, SW31 SW_Push, SW32 SW_Push, SW33 SW_Push, SW34 SW_Push, SW35 SW_Push, SW36 SW_Push, SW37 SW_Push, SW38 SW_Push, SW39 SW_Push, SW4 SW_Push, SW40 SW_Push, SW41 SW_Push, SW42 SW_Push, SW43 SW_Push, SW44 SW_Push, SW45 SW_Push, SW46 SW_Push, SW47 SW_Push, SW48 SW_Push, SW49 SW_Push, SW5 SW_Push, SW50 SW_Push, SW51 SW_Push, SW52 SW_Push, SW53 SW_Push, SW54 SW_Push, SW55 SW_Push, SW56 SW_Push, SW57 SW_Push, SW58 SW_Push, SW59 SW_Push, SW6 SW_Push, SW60 SW_Push, SW61 SW_Push, SW62 SW_Push, SW63 SW_Push, SW64 SW_Push, SW65 SW_Push, SW66 SW_Push, SW67 SW_Push, SW68 SW_Push, SW69 SW_Push, SW7 SW_Push, SW70 SW_Push, SW71 SW_Push, SW72 SW_Push, SW73 SW_Push, SW74 SW_Push, SW75 SW_Push, SW76 SW_Push, SW77 SW_Push, SW78 SW_Push, SW79 SW_Push, SW8 SW_Push, SW80 SW_Push, SW81 SW_Push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

Commit message: Pour GND on both copper layers, stitched with 122 vias
F.Cu and B.Cu each get a GND zone (the Pico's GND net) over the whole
outline: 0.3 mm clearance, thermal reliefs, island removal always. The
matrix slices the pours into strips (columns on F.Cu, rows on B.Cu), so
122 stitching vias, one per key unit where both sides have room, join
them through to the Pico. GND covers 89% of F.Cu and 87% of B.Cu; only
13 slivers under 0.7 mm2 are dropped.

fab/ground_pour.py generated the pours and vias and replaces them when
rerun after rerouting.

Co-Authored-By: Claude Opus 5.5 <noreply@anthropic.com>
Routing:
- net Net-(U1-GND-Pad13): vias 0 -> 122
- added copper zone on B.Cu, net Net-(U1-GND-Pad13)
- added copper zone on F.Cu, net Net-(U1-GND-Pad13)

Commit message: Bump the board to v0.3 and drop the name from the F.Silk legend
The F.Silk legend now reads "alps75-zug - v0.3 - 2026" (was "alps75-zug -
v0.2 - Bert Vidal - 2026"). It was changed through KiCad 10.0.6's Python
API so the Arial Black render cache matches the new text; it keeps its
left-bottom anchor, so it is 12.7 mm shorter.

The board and schematic title blocks also get rev "0.3", so the fab
outputs carry the revision in their X2 ProjectId instead of "rev?".

Co-Authored-By: Claude Opus 5.5 <noreply@anthropic.com>
Other:
- board text added: "alps75-zug - v0.3 - 2026"
- board text removed: "alps75-zug - v0.2 - Bert Vidal - 2026"
